Commit message: still on meshes

File: vision_bot/urdf/vision_rpi_bot.urdf (robot description, URDF)
Before this commit: robot vision_rpi_bot, 1 links, 0 joints
Links:
- link base_link: geometry collision mesh filename=package://vision_bot/meshes/base.dae; visual mesh filename=package://ros_2_vision_tutorial/vision_bot/meshes/base.dae

Commit message: urdf updated

File: vision_bot/urdf/vision_rpi_bot.urdf (robot description, URDF)
Before this commit: robot vision_rpi_bot, 1 links, 0 joints
Links:
- added link base_footprint
- added link camera_link, mass 0.75; collision mesh filename=package://vision_bot/meshes/rpi_camera.dae; visual mesh filename=package://vision_bot/meshes/rpi_camera.dae
- added link caster_holder_link, mass 0.1; collision mesh filename=package://vision_bot/meshes/caster_holder.dae; visual mesh filename=package://vision_bot/meshes/caster_holder.dae
- added link caster_wheel_link, mass 0.1; collision mesh filename=package://vision_bot/meshes/caster_wheel.dae; visual mesh filename=package://vision_bot/meshes/caster_wheel.dae
- added link cover_link, mass 0.5; collision mesh filename=package://vision_bot/meshes/cover.dae; visual mesh filename=package://vision_bot/meshes/cover.dae
- added link lidar_link
- added link wheel_left_link, mass 1; collision mesh filename=package://vision_bot/meshes/wheel.dae; visual mesh filename=package://vision_bot/meshes/wheel.dae
- added link wheel_right_link, mass 1; collision mesh filename=package://vision_bot/meshes/wheel.dae; visual mesh filename=package://vision_bot/meshes/wheel.dae
- link base_link: geometry collision mesh filename=package://vision_bot/meshes/base.dae; visual mesh filename=package://vision_bot/meshes/base.dae
Joints:
- added joint base_joint: type fixed, parent base_footprint, child base_link, origin xyz=0 0 0.14 rpy=0 0 0
- added joint camera_joint: type fixed, parent base_link, child camera_link, origin xyz=0 -0.18 0.2 rpy=0.0 0 -1.57
- added joint caster_holder_joint: type continuous, parent base_link, child caster_holder_link, origin xyz=0 -0.19 -0.015 rpy=0.0 0.0 0.0, axis 0 0 1
- added joint caster_wheel_joint: type continuous, parent caster_holder_link, child caster_wheel_link, origin xyz=0 -0.003  -0.086 rpy=0.0 0.0 0.0, axis 1 0 0
- added joint cover_joint: type fixed, parent base_link, child cover_link, origin xyz=0.0015  0 0.08 rpy=0 0 0
- added joint lidar_joint: type fixed, parent base_link, child lidar_link, origin xyz=0 -0.25 0.1 rpy=0.0 0 -3.14
- added joint wheel_left_joint: type continuous, parent base_link, child wheel_left_link, origin xyz=0.233  0.14 -0.045   rpy=0 0.0 -1.57, axis 0.0 1 0
- added joint wheel_right_joint: type continuous, parent base_link, child wheel_right_link, origin xyz=-0.232  0.14 -0.045   rpy=0 0.0 -1.57, axis 0 1 0
